Commit message: Add nadir camera

File: pud_description/urdf/component_snippets.xacro (robot description, xacro)
@@ -18,5 +18,6 @@
 <robot xmlns:xacro="http://ros.org/wiki/xacro">
   <!-- Macro to add logging to a bag file. -->
-  <xacro:macro name="bag_plugin_macro" params="namespace bag_file rotor_velocity_slowdown_sim wait_to_record_bag">
+  <xacro:macro name="bag_plugin_macro"
+    params="namespace bag_file rotor_velocity_slowdown_sim wait_to_record_bag">
     <gazebo>
       <plugin filename="librotors_gazebo_bag_plugin.so" name="rosbag">
@@ -31,5 +32,6 @@
   </xacro:macro>
   <!-- Macro to add a camera. -->
-  <xacro:macro name="camera_macro" params="namespace parent_link camera_suffix frame_rate
+  <xacro:macro name="camera_macro"
+    params="namespace parent_link camera_suffix frame_rate
       horizontal_fov image_width image_height image_format min_distance
       max_distance noise_mean noise_stddev enable_visual *geometry *origin">
@@ -47,5 +49,5 @@
             <xacro:insert_block name="geometry" />
           </geometry>
-          <material name="red" />
+          <material name="black" />
         </visual>
       </xacro:if>
@@ -90,5 +92,6 @@
           </noise>
         </camera>
-        <plugin name="${namespace}_camera_${camera_suffix}_controller" filename="libgazebo_ros_camera.so">
+        <plugin name="${namespace}_camera_${camera_suffix}_controller"
+          filename="libgazebo_ros_camera.so">
           <robotNamespace>${namespace}</robotNamespace>
           <alwaysOn>true</alwaysOn>
@@ -110,5 +113,6 @@
   <!-- Camera joint macro - just the joints, links, and collisions for a single
        camera. -->
-  <xacro:macro name="camera_joint_macro" params="namespace parent_link camera_suffix enable_visual *origin *geometry">
+  <xacro:macro name="camera_joint_macro"
+    params="namespace parent_link camera_suffix enable_visual *origin *geometry">
     <link name="${namespace}/camera_${camera_suffix}_link">
       <collision>
@@ -140,5 +144,6 @@
   </xacro:macro>
   <!-- Camera sensor macro - just image parameters. -->
-  <xacro:macro name="camera_sensor_macro" params="camera_suffix horizontal_fov image_width image_height
+  <xacro:macro name="camera_sensor_macro"
+    params="camera_suffix horizontal_fov image_width image_height
       image_format min_distance max_distance noise_mean noise_stddev
       baseline">
@@ -166,5 +171,6 @@
   </xacro:macro>
   <!-- Macro to add a multicamera (stereo pair). -->
-  <xacro:macro name="stereo_camera_macro" params="namespace camera_name parent_link frame_rate
+  <xacro:macro name="stereo_camera_macro"
+    params="namespace camera_name parent_link frame_rate
       horizontal_fov image_width image_height image_format min_distance
       max_distance noise_mean noise_stddev enable_visual origin_offset_x
@@ -172,9 +178,11 @@
     <!-- These are parameters for the left camera link and then the right
         as well. -->
-    <xacro:camera_joint_macro namespace="${namespace}" parent_link="${parent_link}" camera_suffix="left" enable_visual="${enable_visual}">
+    <xacro:camera_joint_macro namespace="${namespace}" parent_link="${parent_link}"
+      camera_suffix="left" enable_visual="${enable_visual}">
       <origin xyz="${origin_offset_x} ${baseline_y/2} ${origin_offset_z}" rpy="0 0 0" />
       <xacro:insert_block name="geometry" />
     </xacro:camera_joint_macro>
-    <xacro:camera_joint_macro namespace="${namespace}" parent_link="${parent_link}" camera_suffix="right" enable_visual="${enable_visual}">
+    <xacro:camera_joint_macro namespace="${namespace}" parent_link="${parent_link}"
+      camera_suffix="right" enable_visual="${enable_visual}">
       <origin xyz="${origin_offset_x} ${-baseline_y/2} ${origin_offset_z}" rpy="0 0 0" />
       <xacro:insert_block name="geometry" />
@@ -191,7 +199,13 @@
         <update_rate>${frame_rate}</update_rate>
         <!-- Here we set up the individual cameras of the stereo head. -->
-        <xacro:camera_sensor_macro camera_suffix="left" horizontal_fov="${horizontal_fov}" image_width="${image_width}" image_height="${image_height}" image_format="${image_format}" min_distance="${min_distance}" max_distance="${max_distance}" noise_mean="${noise_mean}" noise_stddev="${noise_stddev}" baseline="0">
+        <xacro:camera_sensor_macro camera_suffix="left" horizontal_fov="${horizontal_fov}"
+          image_width="${image_width}" image_height="${image_height}" image_format="${image_format}"
+          min_distance="${min_distance}" max_distance="${max_distance}" noise_mean="${noise_mean}"
+          noise_stddev="${noise_stddev}" baseline="0">
         </xacro:camera_sensor_macro>
-        <xacro:camera_sensor_macro camera_suffix="right" horizontal_fov="${horizontal_fov}" image_width="${image_width}" image_height="${image_height}" image_format="${image_format}" min_distance="${min_distance}" max_distance="${max_distance}" noise_mean="${noise_mean}" noise_stddev="${noise_stddev}" baseline="${baseline_y}">
+        <xacro:camera_sensor_macro camera_suffix="right" horizontal_fov="${horizontal_fov}"
+          image_width="${image_width}" image_height="${image_height}" image_format="${image_format}"
+          min_distance="${min_distance}" max_distance="${max_distance}" noise_mean="${noise_mean}"
+          noise_stddev="${noise_stddev}" baseline="${baseline_y}">
         </xacro:camera_sensor_macro>
         <!-- Stereo controller, setting the transforms between the two cameras. -->
@@ -239,5 +253,6 @@
   <!-- ================== MAVLINK INTERFACE MACRO ==================== -->
   <!-- =============================================================== -->
-  <xacro:macro name="mavlink_interface_macro" params="namespace mavlink_sub_topic imu_sub_topic mavlink_pub_topic
+  <xacro:macro name="mavlink_interface_macro"
+    params="namespace mavlink_sub_topic imu_sub_topic mavlink_pub_topic
       motors_speeds_pub_topic gps_update_freq rotor_count reference_magnetic_field_north
       reference_magnetic_field_east reference_magnetic_field_down reference_latitude
@@ -252,5 +267,6 @@
         <gpsUpdateFreq>${gps_update_freq}</gpsUpdateFreq>        <!-- Frequency of HIL GPS messages [Hz] -->
         <rotorCount>${rotor_count}</rotorCount>
-        <!-- [Gauss] Below are the North, East, and Down components of the Earth's magnetic field at the reference location.
+        <!-- [Gauss] Below are the North, East, and Down components of the Earth's magnetic field at
+        the reference location.
              The default reference location is Zurich (lat=+47.3667degN, lon=+8.5500degE, h=+500m, WGS84).
 	     You can obtain the magnetic field strength for your location using the World Magnetic Model:
@@ -259,6 +275,8 @@
         <referenceMagEast>${reference_magnetic_field_east}</referenceMagEast>
         <referenceMagDown>${reference_magnetic_field_down}</referenceMagDown>
-        <referenceLatitude>${reference_latitude}</referenceLatitude>        <!-- the initial latitude [degrees [-90, 90]] -->
-        <referenceLongitude>${reference_longitude}</referenceLongitude>        <!-- the initial longitude [degrees [-180, 180]] -->
+        <referenceLatitude>${reference_latitude}</referenceLatitude>        <!-- the initial latitude
+        [degrees [-90, 90]] -->
+        <referenceLongitude>${reference_longitude}</referenceLongitude>        <!-- the initial longitude
+        [degrees [-180, 180]] -->
         <referenceAltitude>${reference_altitude}</referenceAltitude>        <!-- the initial altitude [m] -->
       </plugin>
@@ -266,5 +284,6 @@
   </xacro:macro>
   <!-- Macro to add an IMU. -->
-  <xacro:macro name="imu_plugin_macro" params="namespace imu_suffix parent_link imu_topic
+  <xacro:macro name="imu_plugin_macro"
+    params="namespace imu_suffix parent_link imu_topic
       mass_imu_sensor gyroscope_noise_density gyroscope_random_walk
       gyroscope_bias_correlation_time gyroscope_turn_on_bias_sigma
@@ -292,20 +311,32 @@
         <!-- A good description of the IMU parameters can be found in the kalibr documentation:
            https://github.com/ethz-asl/kalibr/wiki/IMU-Noise-Model-and-Intrinsics -->
-        <robotNamespace>${namespace}</robotNamespace>        <!-- (string, required): ros namespace in which the messages are published -->
-        <linkName>${namespace}/imu${imu_suffix}_link</linkName>        <!-- (string, required): name of the body which holds the IMU sensor -->
-        <imuTopic>${imu_topic}</imuTopic>        <!-- (string): name of the sensor output topic and prefix of service names (defaults to imu) -->
-        <gyroscopeNoiseDensity>${gyroscope_noise_density}</gyroscopeNoiseDensity>        <!-- Gyroscope noise density (two-sided spectrum) [rad/s/sqrt(Hz)] -->
-        <gyroscopeRandomWalk>${gyroscope_random_walk}</gyroscopeRandomWalk>        <!-- Gyroscope bias random walk [rad/s/s/sqrt(Hz)] -->
-        <gyroscopeBiasCorrelationTime>${gyroscope_bias_correlation_time}</gyroscopeBiasCorrelationTime>        <!-- Gyroscope bias correlation time constant [s] -->
-        <gyroscopeTurnOnBiasSigma>${gyroscope_turn_on_bias_sigma}</gyroscopeTurnOnBiasSigma>        <!-- Gyroscope turn on bias standard deviation [rad/s] -->
-        <accelerometerNoiseDensity>${accelerometer_noise_density}</accelerometerNoiseDensity>        <!-- Accelerometer noise density (two-sided spectrum) [m/s^2/sqrt(Hz)] -->
-        <accelerometerRandomWalk>${accelerometer_random_walk}</accelerometerRandomWalk>        <!-- Accelerometer bias random walk. [m/s^2/s/sqrt(Hz)] -->
-        <accelerometerBiasCorrelationTime>${accelerometer_bias_correlation_time}</accelerometerBiasCorrelationTime>        <!-- Accelerometer bias correlation time constant [s] -->
-        <accelerometerTurnOnBiasSigma>${accelerometer_turn_on_bias_sigma}</accelerometerTurnOnBiasSigma>        <!-- Accelerometer turn on bias standard deviation [m/s^2] -->
+        <robotNamespace>${namespace}</robotNamespace>        <!-- (string, required): ros namespace in which
+        the messages are published -->
+        <linkName>${namespace}/imu${imu_suffix}_link</linkName>        <!-- (string, required): name of the
+        body which holds the IMU sensor -->
+        <imuTopic>${imu_topic}</imuTopic>        <!-- (string): name of the sensor output topic and prefix
+        of service names (defaults to imu) -->
+        <gyroscopeNoiseDensity>${gyroscope_noise_density}</gyroscopeNoiseDensity>        <!-- Gyroscope
+        noise density (two-sided spectrum) [rad/s/sqrt(Hz)] -->
+        <gyroscopeRandomWalk>${gyroscope_random_walk}</gyroscopeRandomWalk>        <!-- Gyroscope bias
+        random walk [rad/s/s/sqrt(Hz)] -->
+        <gyroscopeBiasCorrelationTime>${gyroscope_bias_correlation_time}</gyroscopeBiasCorrelationTime>        <!--
+        Gyroscope bias correlation time constant [s] -->
+        <gyroscopeTurnOnBiasSigma>${gyroscope_turn_on_bias_sigma}</gyroscopeTurnOnBiasSigma>        <!--
+        Gyroscope turn on bias standard deviation [rad/s] -->
+        <accelerometerNoiseDensity>${accelerometer_noise_density}</accelerometerNoiseDensity>        <!--
+        Accelerometer noise density (two-sided spectrum) [m/s^2/sqrt(Hz)] -->
+        <accelerometerRandomWalk>${accelerometer_random_walk}</accelerometerRandomWalk>        <!--
+        Accelerometer bias random walk. [m/s^2/s/sqrt(Hz)] -->
+        <accelerometerBiasCorrelationTime>${accelerometer_bias_correlation_time}</accelerometerBiasCorrelationTime>        <!--
+        Accelerometer bias correlation time constant [s] -->
+        <accelerometerTurnOnBiasSigma>${accelerometer_turn_on_bias_sigma}</accelerometerTurnOnBiasSigma>        <!--
+        Accelerometer turn on bias standard deviation [m/s^2] -->
       </plugin>
     </gazebo>
   </xacro:macro>
   <!-- Macro to add a generic odometry sensor. -->
-  <xacro:macro name="odometry_plugin_macro" params="
+  <xacro:macro name="odometry_plugin_macro"
+    params="
       namespace odometry_sensor_suffix parent_link pose_topic pose_with_covariance_topic
       position_topic transform_topic odometry_topic parent_frame_id child_frame_id
@@ -332,5 +363,6 @@
     </joint>
     <gazebo>
-      <plugin filename="librotors_gazebo_odometry_plugin.so" name="odometry_sensor${odometry_sensor_suffix}">
+      <plugin filename="librotors_gazebo_odometry_plugin.so"
+        name="odometry_sensor${odometry_sensor_suffix}">
         <linkName>${namespace}/odometry_sensor${odometry_sensor_suffix}_link</linkName>
         <robotNamespace>${namespace}</robotNamespace>
@@ -340,20 +372,35 @@
         <transformTopic>${transform_topic}</transformTopic>
         <odometryTopic>${odometry_topic}</odometryTopic>
-        <parentFrameId>${parent_frame_id}</parentFrameId>        <!-- Use the scoped link name here. e.g. Model::link. -->
+        <parentFrameId>${parent_frame_id}</parentFrameId>        <!-- Use the scoped link name here. e.g.
+        Model::link. -->
         <childFrameId>${child_frame_id}</childFrameId>
-        <measurementDivisor>${measurement_divisor}</measurementDivisor>        <!-- only every (seq % measurementDivisor) == 0 measurement is published [int] -->
-        <measurementDelay>${measurement_delay}</measurementDelay>        <!-- time that measurement gets held back before it's published in [simulation cycles (int)] -->
-        <unknownDelay>${unknown_delay}</unknownDelay>        <!-- additional delay, that just gets added to the timestamp [s] -->
-        <noiseNormalPosition>${noise_normal_position}</noiseNormalPosition>        <!-- standard deviation of additive white gaussian noise [m] -->
-        <noiseNormalQuaternion>${noise_normal_quaternion}</noiseNormalQuaternion>        <!-- standard deviation white gaussian noise [rad]: q_m = q*quaternionFromSmallAngleApproximation(noiseNormalQ) -->
-        <noiseNormalLinearVelocity>${noise_normal_linear_velocity}</noiseNormalLinearVelocity>        <!-- standard deviation of additive white gaussian noise [m/s] -->
-        <noiseNormalAngularVelocity>${noise_normal_angular_velocity}</noiseNormalAngularVelocity>        <!-- standard deviation of additive white gaussian noise [rad/s] -->
-        <noiseUniformPosition>${noise_uniform_position}</noiseUniformPosition>        <!-- symmetric bounds of uniform noise [m] -->
-        <noiseUniformQuaternion>${noise_uniform_quaternion}</noiseUniformQuaternion>        <!-- symmetric bounds of uniform noise [rad], computation see above -->
-        <noiseUniformLinearVelocity>${noise_uniform_linear_velocity}</noiseUniformLinearVelocity>        <!-- symmetric bounds of uniform noise [m/s] -->
-        <noiseUniformAngularVelocity>${noise_uniform_angular_velocity}</noiseUniformAngularVelocity>        <!-- symmetric bounds of uniform noise [rad/s] -->
+        <measurementDivisor>${measurement_divisor}</measurementDivisor>        <!-- only every (seq %
+        measurementDivisor) == 0 measurement is published [int] -->
+        <measurementDelay>${measurement_delay}</measurementDelay>        <!-- time that measurement gets
+        held back before it's published in [simulation cycles (int)] -->
+        <unknownDelay>${unknown_delay}</unknownDelay>        <!-- additional delay, that just gets added to
+        the timestamp [s] -->
+        <noiseNormalPosition>${noise_normal_position}</noiseNormalPosition>        <!-- standard deviation
+        of additive white gaussian noise [m] -->
+        <noiseNormalQuaternion>${noise_normal_quaternion}</noiseNormalQuaternion>        <!-- standard
+        deviation white gaussian noise [rad]: q_m =
+        q*quaternionFromSmallAngleApproximation(noiseNormalQ) -->
+        <noiseNormalLinearVelocity>${noise_normal_linear_velocity}</noiseNormalLinearVelocity>        <!--
+        standard deviation of additive white gaussian noise [m/s] -->
+        <noiseNormalAngularVelocity>${noise_normal_angular_velocity}</noiseNormalAngularVelocity>        <!--
+        standard deviation of additive white gaussian noise [rad/s] -->
+        <noiseUniformPosition>${noise_uniform_position}</noiseUniformPosition>        <!-- symmetric bounds
+        of uniform noise [m] -->
+        <noiseUniformQuaternion>${noise_uniform_quaternion}</noiseUniformQuaternion>        <!-- symmetric
+        bounds of uniform noise [rad], computation see above -->
+        <noiseUniformLinearVelocity>${noise_uniform_linear_velocity}</noiseUniformLinearVelocity>        <!--
+        symmetric bounds of uniform noise [m/s] -->
+        <noiseUniformAngularVelocity>${noise_uniform_angular_velocity}</noiseUniformAngularVelocity>        <!--
+        symmetric bounds of uniform noise [rad/s] -->
         <xacro:if value="${enable_odometry_map}">
-          <covarianceImage>package://pud_gazebo/resource/${odometry_map}</covarianceImage>          <!-- a bitmap image describing where the sensor works (white), and where not (black) -->
-          <covarianceImageScale>${image_scale}</covarianceImageScale>          <!-- the scale of the image in the gazebo world, if set to 1.0, 1 pixel in the image corresponds to 1 meter in the world -->
+          <covarianceImage>package://pud_gazebo/resource/${odometry_map}</covarianceImage>          <!-- a
+          bitmap image describing where the sensor works (white), and where not (black) -->
+          <covarianceImageScale>${image_scale}</covarianceImageScale>          <!-- the scale of the image in
+          the gazebo world, if set to 1.0, 1 pixel in the image corresponds to 1 meter in the world -->
         </xacro:if>
       </plugin>
@@ -361,5 +408,6 @@
   </xacro:macro>
   <!-- Macro to add a GPS sensor. -->
-  <xacro:macro name="gps_plugin_macro" params="namespace gps_suffix parent_link gps_topic ground_speed_topic
+  <xacro:macro name="gps_plugin_macro"
+    params="namespace gps_suffix parent_link gps_topic ground_speed_topic
       mass_gps_sensor horizontal_pos_std_dev vertical_pos_std_dev
       horizontal_vel_std_dev vertical_vel_std_dev *inertia *origin">
@@ -424,13 +472,22 @@
           </velocity_sensing>
         </gps>
-        <plugin filename="librotors_gazebo_gps_plugin.so" name="rotors_gazebo_gps${gps_suffix}_plugin">
-          <robotNamespace>${namespace}</robotNamespace>          <!-- (string, required): ros namespace in which the messages are published -->
-          <linkName>${namespace}/gps${gps_suffix}_link</linkName>          <!-- (string, required): name of the body which holds the GPS sensor -->
-          <gpsTopic>${gps_topic}</gpsTopic>          <!-- (string): name of the sensor output topic and prefix of service names (defaults to 'gps') -->
-          <groundSpeedTopic>${ground_speed_topic}</groundSpeedTopic>          <!-- (string): name of the ground speed output topic (defaults to 'ground_speed') -->
-          <horPosStdDev>${horizontal_pos_std_dev}</horPosStdDev>          <!-- standard deviation for horizontal position noise [m] -->
-          <verPosStdDev>${vertical_pos_std_dev}</verPosStdDev>          <!-- standard deviation for vertical position noise [m] -->
-          <horVelStdDev>${horizontal_vel_std_dev}</horVelStdDev>          <!-- standard deviation for horizontal speed noise [m/s] -->
-          <verVelStdDev>${vertical_vel_std_dev}</verVelStdDev>          <!-- standard deviation for vertical speed noise [m/s] -->
+        <plugin filename="librotors_gazebo_gps_plugin.so"
+          name="rotors_gazebo_gps${gps_suffix}_plugin">
+          <robotNamespace>${namespace}</robotNamespace>          <!-- (string, required): ros namespace in
+          which the messages are published -->
+          <linkName>${namespace}/gps${gps_suffix}_link</linkName>          <!-- (string, required): name of
+          the body which holds the GPS sensor -->
+          <gpsTopic>${gps_topic}</gpsTopic>          <!-- (string): name of the sensor output topic and prefix
+          of service names (defaults to 'gps') -->
+          <groundSpeedTopic>${ground_speed_topic}</groundSpeedTopic>          <!-- (string): name of the
+          ground speed output topic (defaults to 'ground_speed') -->
+          <horPosStdDev>${horizontal_pos_std_dev}</horPosStdDev>          <!-- standard deviation for
+          horizontal position noise [m] -->
+          <verPosStdDev>${vertical_pos_std_dev}</verPosStdDev>          <!-- standard deviation for vertical
+          position noise [m] -->
+          <horVelStdDev>${horizontal_vel_std_dev}</horVelStdDev>          <!-- standard deviation for
+          horizontal speed noise [m/s] -->
+          <verVelStdDev>${vertical_vel_std_dev}</verVelStdDev>          <!-- standard deviation for vertical
+          speed noise [m/s] -->
         </plugin>
       </sensor>
@@ -438,5 +495,6 @@
   </xacro:macro>
   <!-- Macro to add a magnetometer. -->
-  <xacro:macro name="magnetometer_plugin_macro" params="namespace magnetometer_suffix parent_link magnetometer_topic
+  <xacro:macro name="magnetometer_plugin_macro"
+    params="namespace magnetometer_suffix parent_link magnetometer_topic
       mass_magnetometer_sensor ref_mag_north ref_mag_east ref_mag_down
       noise_normal noise_uniform_initial_bias *inertia *origin">
@@ -458,9 +516,14 @@
     </joint>
     <gazebo>
-      <plugin filename="librotors_gazebo_magnetometer_plugin.so" name="rotors_gazebo_magnetometer${magnetometer_suffix}_plugin">
-        <robotNamespace>${namespace}</robotNamespace>        <!-- (string, required): ros namespace in which the messages are published -->
-        <linkName>${namespace}/magnetometer${magnetometer_suffix}_link</linkName>        <!-- (string, required): name of the body which holds the magnetometer -->
-        <magnetometerTopic>${magnetometer_topic}</magnetometerTopic>        <!-- (string): name of the sensor output topic and prefix of service names (defaults to 'magnetic_field') -->
-        <!-- [Tesla] Below is the reference Earth's magnetic field at the reference location in NED frame.
+      <plugin filename="librotors_gazebo_magnetometer_plugin.so"
+        name="rotors_gazebo_magnetometer${magnetometer_suffix}_plugin">
+        <robotNamespace>${namespace}</robotNamespace>        <!-- (string, required): ros namespace in which
+        the messages are published -->
+        <linkName>${namespace}/magnetometer${magnetometer_suffix}_link</linkName>        <!-- (string,
+        required): name of the body which holds the magnetometer -->
+        <magnetometerTopic>${magnetometer_topic}</magnetometerTopic>        <!-- (string): name of the
+        sensor output topic and prefix of service names (defaults to 'magnetic_field') -->
+        <!-- [Tesla] Below is the reference Earth's magnetic field at the reference location in NED
+        frame.
              The default reference location is Zurich (lat=+47.3667degN, lon=+8.5500degE, h=+500m, WGS84).
 	     You can obtain the magnetic field strength for your location using the World Magnetic Model:
@@ -469,11 +532,14 @@
         <refMagEast>${ref_mag_east}</refMagEast>
         <refMagDown>${ref_mag_down}</refMagDown>
-        <noiseNormal>${noise_normal}</noiseNormal>        <!-- standard deviation of additive white gaussian noise [Tesla] -->
-        <noiseUniformInitialBias>${noise_uniform_initial_bias}</noiseUniformInitialBias>        <!-- symmetric bounds of uniform noise for initial sensor bias [Tesla] -->
+        <noiseNormal>${noise_normal}</noiseNormal>        <!-- standard deviation of additive white gaussian
+        noise [Tesla] -->
+        <noiseUniformInitialBias>${noise_uniform_initial_bias}</noiseUniformInitialBias>        <!--
+        symmetric bounds of uniform noise for initial sensor bias [Tesla] -->
       </plugin>
     </gazebo>
   </xacro:macro>
   <!-- Macro to add an air pressure sensor. -->
-  <xacro:macro name="pressure_sensor_plugin_macro" params="namespace pressure_sensor_suffix parent_link pressure_topic
+  <xacro:macro name="pressure_sensor_plugin_macro"
+    params="namespace pressure_sensor_suffix parent_link pressure_topic
       mass_pressure_sensor reference_altitude pressure_variance *inertia
       *origin">
@@ -495,15 +561,21 @@
     </joint>
     <gazebo>
-      <plugin filename="librotors_gazebo_pressure_plugin.so" name="rotors_gazebo_pressure_sensor${pressure_sensor_suffix}_plugin">
-        <robotNamespace>${namespace}</robotNamespace>        <!-- (string, required): ros namespace in which the messages are published -->
-        <linkName>${namespace}/pressure_sensor${pressure_sensor_suffix}_link</linkName>        <!-- (string, required): name of the body which holds the pressure sensor -->
-        <pressureTopic>${pressure_topic}</pressureTopic>        <!-- (string): name of the sensor output topic and prefix of service names (defaults to 'air_pressure') -->
+      <plugin filename="librotors_gazebo_pressure_plugin.so"
+        name="rotors_gazebo_pressure_sensor${pressure_sensor_suffix}_plugin">
+        <robotNamespace>${namespace}</robotNamespace>        <!-- (string, required): ros namespace in which
+        the messages are published -->
+        <linkName>${namespace}/pressure_sensor${pressure_sensor_suffix}_link</linkName>        <!-- (string,
+        required): name of the body which holds the pressure sensor -->
+        <pressureTopic>${pressure_topic}</pressureTopic>        <!-- (string): name of the sensor output
+        topic and prefix of service names (defaults to 'air_pressure') -->
         <referenceAltitude>${reference_altitude}</referenceAltitude>        <!-- the initial altitude [m] -->
-        <pressureVariance>${pressure_variance}</pressureVariance>        <!-- the air pressure variance [Pa^2] -->
+        <pressureVariance>${pressure_variance}</pressureVariance>        <!-- the air pressure variance
+        [Pa^2] -->
       </plugin>
     </gazebo>
   </xacro:macro>
   <!-- Macro to add the wind plugin. -->
-  <xacro:macro name="wind_plugin_macro" params="namespace xyz_offset wind_direction wind_force_mean
+  <xacro:macro name="wind_plugin_macro"
+    params="namespace xyz_offset wind_direction wind_force_mean
       wind_gust_direction wind_gust_duration wind_gust_start
       wind_gust_force_mean wind_speed_mean use_custom_static_wind_field
@@ -529,6 +601,10 @@
   <!-- VI sensor macros -->
   <!-- Macro to add a VI-sensor camera. -->
-  <xacro:macro name="vi_sensor_camera_macro" params="namespace parent_link camera_suffix frame_rate *origin">
-    <xacro:camera_macro namespace="${namespace}" parent_link="${parent_link}" camera_suffix="${camera_suffix}" frame_rate="${frame_rate}" horizontal_fov="1.3962634" image_width="752" image_height="480" image_format="L8" min_distance="0.02" max_distance="30" noise_mean="0.0" noise_stddev="0.007" enable_visual="true">
+  <xacro:macro name="vi_sensor_camera_macro"
+    params="namespace parent_link camera_suffix frame_rate *origin">
+    <xacro:camera_macro namespace="${namespace}" parent_link="${parent_link}"
+      camera_suffix="${camera_suffix}" frame_rate="${frame_rate}" horizontal_fov="1.3962634"
+      image_width="752" image_height="480" image_format="L8" min_distance="0.02" max_distance="30"
+      noise_mean="0.0" noise_stddev="0.007" enable_visual="true">
       <mesh filename="package://pud_description/meshes/vi_camera.dae" scale="1 1 1" />
       <xacro:insert_block name="origin" />
@@ -536,11 +612,18 @@
   </xacro:macro>
   <!-- Macro to add a VI-sensor stereo camera. -->
-  <xacro:macro name="vi_sensor_stereo_camera_macro" params="namespace parent_link frame_rate origin_offset_x baseline_y origin_offset_z max_range">
-    <xacro:stereo_camera_macro namespace="${namespace}" camera_name="vi_sensor" parent_link="${parent_link}" frame_rate="${frame_rate}" horizontal_fov="1.3962634" image_width="752" image_height="480" image_format="L8" min_distance="0.02" max_distance="${max_range}" noise_mean="0.0" noise_stddev="0.007" enable_visual="false" origin_offset_x="${origin_offset_x}" baseline_y="${baseline_y}" origin_offset_z="${origin_offset_z}">
+  <xacro:macro name="vi_sensor_stereo_camera_macro"
+    params="namespace parent_link frame_rate origin_offset_x baseline_y origin_offset_z max_range">
+    <xacro:stereo_camera_macro namespace="${namespace}" camera_name="vi_sensor"
+      parent_link="${parent_link}" frame_rate="${frame_rate}" horizontal_fov="1.3962634"
+      image_width="752" image_height="480" image_format="L8" min_distance="0.02"
+      max_distance="${max_range}" noise_mean="0.0" noise_stddev="0.007" enable_visual="false"
+      origin_offset_x="${origin_offset_x}" baseline_y="${baseline_y}"
+      origin_offset_z="${origin_offset_z}">
       <cylinder length="0.01" radius="0.007" />
     </xacro:stereo_camera_macro>
   </xacro:macro>
   <!-- Macro to add a depth camera on the VI-sensor. -->
-  <xacro:macro name="vi_sensor_depth_macro" params="namespace parent_link camera_suffix frame_rate max_range *origin">
+  <xacro:macro name="vi_sensor_depth_macro"
+    params="namespace parent_link camera_suffix frame_rate max_range *origin">
     <link name="${namespace}/camera_${camera_suffix}_link">
       <collision>
@@ -610,5 +693,6 @@
   </xacro:macro>
   <!-- VI-Sensor Macro -->
-  <xacro:macro name="vi_sensor_macro" params="namespace parent_link enable_cameras enable_depth enable_ground_truth *origin">
+  <xacro:macro name="vi_sensor_macro"
+    params="namespace parent_link enable_cameras enable_depth enable_ground_truth *origin">
     <!-- Vi Sensor Link -->
     <link name="${namespace}/vi_sensor_link">
@@ -639,10 +723,14 @@
     <xacro:if value="${enable_cameras}">
       <!-- Insert stereo pair. -->
-      <xacro:vi_sensor_stereo_camera_macro namespace="${namespace}" parent_link="${namespace}/vi_sensor_link" frame_rate="30.0" origin_offset_x="0.015" baseline_y="${0.055*2}" origin_offset_z="0.0065" max_range="30.0">
+      <xacro:vi_sensor_stereo_camera_macro namespace="${namespace}"
+        parent_link="${namespace}/vi_sensor_link" frame_rate="30.0" origin_offset_x="0.015"
+        baseline_y="${0.055*2}" origin_offset_z="0.0065" max_range="30.0">
       </xacro:vi_sensor_stereo_camera_macro>
     </xacro:if>
     <!-- Depth Sensor -->
     <xacro:if value="${enable_depth}">
-      <xacro:vi_sensor_depth_macro namespace="${namespace}" parent_link="${namespace}/vi_sensor_link" camera_suffix="depth" frame_rate="30.0" max_range="10.0">
+      <xacro:vi_sensor_depth_macro namespace="${namespace}"
+        parent_link="${namespace}/vi_sensor_link" camera_suffix="depth" frame_rate="30.0"
+        max_range="10.0">
         <origin xyz="0.015 0.055 0.0065" rpy="0 0 0" />
       </xacro:vi_sensor_depth_macro>
@@ -651,5 +739,15 @@
     <xacro:if value="${enable_ground_truth}">
       <!-- Odometry Sensor -->
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