Commit message: Add nadir camera

File: pud_description/urdf/iris_base.xacro (robot description, xacro)
@@ -5,4 +5,22 @@
   <!-- Instantiate iris "mechanics" -->
   <xacro:include filename="$(find pud_description)/urdf/iris.xacro" />
+  <xacro:property name="arm_length" value="0.13" />
+  <xacro:camera_macro
+    namespace="${namespace}"
+    parent_link="${namespace}/base_link"
+    camera_suffix="nadir"
+    frame_rate="20.0"
+    horizontal_fov="2"
+    image_width="752"
+    image_height="480"
+    image_format="L8"
+    min_distance="0.02"
+    max_distance="50"
+    noise_mean="0.0"
+    noise_stddev="0.007"
+    enable_visual="true">
+    <box size="0.05 0.05 0.02" />
+    <origin xyz="0 0 ${-arm_length/4}" rpy="0 ${pi/2} 0" />
+  </xacro:camera_macro>
   <!-- Instantiate a controller. -->
   <xacro:controller_plugin_macro namespace="${namespace}" imu_sub_topic="imu" />
@@ -14,9 +32,12 @@
   <xacro:default_imu namespace="${namespace}" parent_link="${namespace}/base_link" />
   <xacro:if value="$(arg enable_ground_truth)">
-    <xacro:ground_truth_imu_and_odometry namespace="${namespace}" parent_link="${namespace}/base_link" />
+    <xacro:ground_truth_imu_and_odometry namespace="${namespace}"
+      parent_link="${namespace}/base_link" />
   </xacro:if>
   <xacro:if value="$(arg enable_logging)">
     <!-- Instantiate a logger -->
-    <xacro:bag_plugin_macro namespace="${namespace}" bag_file="$(arg log_file)" rotor_velocity_slowdown_sim="${rotor_velocity_slowdown_sim}" wait_to_record_bag="$(arg wait_to_record_bag)" />
+    <xacro:bag_plugin_macro namespace="${namespace}" bag_file="$(arg log_file)"
+      rotor_velocity_slowdown_sim="${rotor_velocity_slowdown_sim}"
+      wait_to_record_bag="$(arg wait_to_record_bag)" />
   </xacro:if>
 </robot>
